File: hardware/io-16.kicad_pcb (KiCad board)
At the start: 2 copper layers, 75 x 35 mm, 38 parts, among them J1 AKL_5_2, J10 AKL_5_2, J11 AKL_5_2, J12 AKL_5_2, J13 AKL_5_2, J2 AKL_5_2, J3 AKL_5_2, J4 AKL_5_2, J5 AKL_5_2, J6 AKL_5_2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

Commit message: Add Tinkerforge-CoMCU logo
Parts:
- added G***: LOGO, kicad-libraries:Logo_CoMCU, B.Cu at (128.4, 97.0)
