File: hardware/io16-v2.kicad_pcb (KiCad board)
At the start: 2 copper layers, 75 x 35 mm, 39 parts, among them J1 AKL_5_2, J10 AKL_5_2, J11 AKL_5_2, J12 AKL_5_2, J13 AKL_5_2, J2 AKL_5_2, J3 AKL_5_2, J4 AKL_5_2, J5 AKL_5_2, J6 AKL_5_2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

Commit message: specify processor, fix references
Parts:
- U1: value XMC11XX24 -> XMC1100
Changed lines of the file:
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@@
       (effects (font (size 0.3 0.3) (thickness 0.075)))
     )
-    (fp_text value XMC11XX24 (at 0 0.8 270) (layer F.Fab)
+    (fp_text value XMC1100 (at 0 0.8 270) (layer F.Fab)
       (effects (font (size 0.3 0.3) (thickness 0.075)))
     )
